Commit message: feat: add namespaced three-host bringup and isolation tests

File: src/mycar_description/urdf/car.urdf.xacro (robot description, xacro)
@@ -1,3 +1,5 @@
 <robot name="mycar" xmlns:xacro="http://wiki.ros.org/xacro">
+    <xacro:arg name="prefix" default="" />
+    <xacro:property name="prefix" value="$(arg prefix)" />
     <xacro:include filename="car_base.urdf.xacro" />
     <xacro:include filename="car_laser.urdf.xacro" />

File: src/mycar_description/urdf/car_base.urdf.xacro (robot description, xacro)
@@ -53,5 +53,5 @@
     <xacro:property name="footprint_radius" value="0.001" />
     <!-- base_footprint 是一个虚拟点，代表机器人中心在地面的投影，通常用于导航堆栈 -->
-    <link name="base_footprint">
+    <link name="${prefix}base_footprint">
         <visual>
             <geometry>
@@ -71,5 +71,5 @@
     <xacro:property name="base_joint_z" value="${base_length / 2 + lidi}" />
     <!-- 机器人主体 link -->
-    <link name="base_link">
+    <link name="${prefix}base_link">
         <visual>
             <geometry>
@@ -91,7 +91,7 @@
     </link>
     <!-- 固定关节：连接 base_footprint 到 base_link -->
-    <joint name="link2footprint" type="fixed">
-        <parent link="base_link" />
-        <child link="base_footprint" />
+    <joint name="${prefix}link2footprint" type="fixed">
+        <parent link="${prefix}base_link" />
+        <child link="${prefix}base_footprint" />
         <!-- 将 base_link 抬高，使得 base_link 的中心位于 base_footprint  -->
         <origin xyz="0 0 -${base_height / 2 + lidi}" rpy="0 0 0" />
@@ -107,5 +107,5 @@
     <xacro:macro name="wheel_func" params="wheel_name flag">
         <!-- flag 取 +1 表示左边，-1 表示右边 -->
-        <link name="${wheel_name}_wheel">
+        <link name="${prefix}${wheel_name}_wheel">
             <visual>
                 <geometry>
@@ -128,7 +128,7 @@
         </link>
         <!-- 轮子关节：连续旋转关节，绕 Y 轴旋转 -->
-        <joint name="${wheel_name}2link" type="continuous">
-            <parent link="base_link" />
-            <child link="${wheel_name}_wheel" />
+        <joint name="${prefix}${wheel_name}2link" type="continuous">
+            <parent link="${prefix}base_link" />
+            <child link="${prefix}${wheel_name}_wheel" />
             <!-- 位置：x=0 (前后)，y=±0.1 (左右轮距)，z 为计算值使轮子接地 -->
             <origin xyz=" -0.05175 ${(half_width - 0.0105) * flag} ${wheel_joint_z}" rpy="0 0 0" />
@@ -145,5 +145,5 @@
     <xacro:macro name="small_wheel_func" params="small_wheel_name flag">
         <!-- flag 取 +1 表示前，-1 表示后 -->
-        <link name="${small_wheel_name}_wheel">
+        <link name="${prefix}${small_wheel_name}_wheel">
             <visual>
                 <geometry>
@@ -156,7 +156,7 @@
             </visual>
         </link>
-        <joint name="${small_wheel_name}2link" type="continuous">
-            <parent link="base_link" />
-            <child link="${small_wheel_name}_wheel" />
+        <joint name="${prefix}${small_wheel_name}2link" type="continuous">
+            <parent link="${prefix}base_link" />
+            <child link="${prefix}${small_wheel_name}_wheel" />
             <!-- 位置：x 前后偏移 ±0.08 m，y=0（中间），z 接地 -->
             <origin xyz="${half_length - 0.032} ${(half_width - 0.0427) * flag} ${small_joint_z}" rpy="0 0 0" />

File: src/mycar_description/urdf/car_camera.urdf.xacro (robot description, xacro)
@@ -6,5 +6,5 @@
     <xacro:property name="joint_camera_y" value="0" />
     <xacro:property name="joint_camera_z" value="${base_length / 2 + camera_height / 2}" />
-    <link name="camera">
+    <link name="${prefix}camera">
         <visual>
             <geometry>
@@ -17,7 +17,7 @@
         </visual>
     </link>
-    <joint name="camera2base" type="fixed">
-        <parent link="base_link" />
-        <child link="camera" />
+    <joint name="${prefix}camera2base" type="fixed">
+        <parent link="${prefix}base_link" />
+        <child link="${prefix}camera" />
         <origin xyz="${joint_camera_x} ${joint_camera_y} ${joint_camera_z}" rpy="0 0 0" />
     </joint>

File: src/mycar_description/urdf/car_laser.urdf.xacro (robot description, xacro)
@@ -32,5 +32,5 @@
     <xacro:property name="joint_laser_z" value="${support_length / 2 + laser_length / 2}" />
     <!-- ================= 支撑柱 link 定义 ================= -->
-    <link name="support">
+    <link name="${prefix}support">
         <visual>
             <geometry>
@@ -46,12 +46,12 @@
     </link>
     <!-- ================= 支撑柱到车体的固定关节 ================= -->
-    <joint name="support2base" type="fixed">
-        <parent link="base_link" />        <!-- 父坐标系为车体 base_link -->
-        <child link="support"/>             <!-- 子坐标系为支撑柱 support -->
+    <joint name="${prefix}support2base" type="fixed">
+        <parent link="${prefix}base_link" />        <!-- 父坐标系为车体 base_link -->
+        <child link="${prefix}support"/>             <!-- 子坐标系为支撑柱 support -->
         <!-- 关节原点相对于 base_link 的位置，由上面计算的 joint_support_* 决定 -->
         <origin xyz="${joint_support_x} ${joint_support_y} ${joint_support_z}" rpy="0 0 0" />
     </joint>
     <!-- ================= 激光雷达 link 定义 ================= -->
-    <link name="laser">
+    <link name="${prefix}laser">
         <visual>
             <geometry>
@@ -66,7 +66,7 @@
     </link>
     <!-- ================= 激光雷达到支撑柱的固定关节 ================= -->
-    <joint name="laser2support" type="fixed">
-        <parent link="support" />           <!-- 父坐标系为支撑柱 support -->
-        <child link="laser"/>                <!-- 子坐标系为激光雷达 laser -->
+    <joint name="${prefix}laser2support" type="fixed">
+        <parent link="${prefix}support" />           <!-- 父坐标系为支撑柱 support -->
+        <child link="${prefix}laser"/>                <!-- 子坐标系为激光雷达 laser -->
         <!-- 关节原点相对于 support 的位置，由 joint_laser_* 决定 -->
         <origin xyz="${joint_laser_x} ${joint_laser_y} ${joint_laser_z}" rpy="0 0 ${PI}" />
