Commit message: feat: finalize support geometry and single-car S pretest

File: src/mycar_description/urdf/car_base.urdf.xacro (robot description, xacro)
@@ -68,6 +68,11 @@
     <xacro:property name="half_length" value="${base_length / 2}" />       <!-- 主体长度的一半 (m) -->
     <xacro:property name="half_width" value="${base_width / 2}" />        <!-- 主体宽度的一半 (m) -->
+    <!--
+      base_link 的平面原点固定在左右驱动轮轴线中点。实测该点位于旧车体
+      几何中心后方 49.69 mm，因此车体几何中心在新 base_link 的 +X 方向。
+    -->
+    <xacro:property name="chassis_center_x" value="0.04969" />
     <!-- 计算 base_link 相对于 base_footprint 的高度：主体一半高度 + 离地间隙 -->
-    <xacro:property name="base_joint_z" value="${base_length / 2 + lidi}" />
+    <xacro:property name="base_joint_z" value="${base_height / 2 + lidi}" />
     <!-- 机器人主体 link -->
     <link name="${prefix}base_link">
@@ -76,5 +81,5 @@
                 <box size="${base_length} ${base_width} ${base_height}"/> <!-- 主体形状：长方体，尺寸与属性一致 -->
             </geometry>
-            <origin xyz="0 0 0" rpy="0 0 0" />              <!-- 圆柱中心位于 link 原点 -->
+            <origin xyz="${chassis_center_x} 0 0" rpy="0 0 0" />
             <material name="baselink_color">
                 <color rgba="1.0 0.5 0.2 1.0" />            <!-- 橙色 -->
@@ -85,8 +90,9 @@
                 <box size="${base_length} ${base_width} ${base_height}"/>
             </geometry>
-            <origin xyz="0.0 0.0 0.0" rpy="0.0 0.0 0.0"/>
+            <origin xyz="${chassis_center_x} 0 0" rpy="0 0 0"/>
         </collision>
         <!-- 设置机器人尺寸、质量 -->
-        <xacro:box_inertial_matrix mass="${base_mass}" lx="0.2035" ly="0.145" lz="0.052" />
+        <xacro:box_inertial_matrix mass="${base_mass}" lx="0.2035" ly="0.145" lz="0.052"
+                                   origin_xyz="${chassis_center_x} 0 0" />
     </link>
     <!-- 固定关节：连接 base_footprint 到 base_link -->
@@ -99,4 +105,5 @@
     <!-- ================= 驱动轮（左右轮）定义 ================= -->
     <xacro:property name="wheel_radius" value="0.0325" />    <!-- 驱动轮半径 (m) -->
+    <xacro:property name="wheel_separation" value="0.114" /> <!-- 实测左右轮轴向中心距 (m) -->
     <xacro:property name="wheel_length" value="0.027" />     <!-- 驱动轮厚度 (m) -->
     <xacro:property name="wheel_mass" value="0.1" />         <!-- 驱动轮质量 (kg) -->
@@ -131,6 +138,6 @@
             <parent link="${prefix}base_link" />
             <child link="${prefix}${wheel_name}_wheel" />
-            <!-- 位置：x=0 (前后)，y=±0.1 (左右轮距)，z 为计算值使轮子接地 -->
-            <origin xyz=" -0.05175 ${(half_width - 0.0105) * flag} ${wheel_joint_z}" rpy="0 0 0" />
+            <!-- base_link 就是左右驱动轮轴线中点，所以驱动轮 x 必须为 0。 -->
+            <origin xyz="0 ${(wheel_separation / 2) * flag} ${wheel_joint_z}" rpy="0 0 0" />
             <axis xyz="0 1 0" />                              <!-- 绕 Y 轴旋转 -->
         </joint>
@@ -160,5 +167,5 @@
             <child link="${prefix}${small_wheel_name}_wheel" />
             <!-- 位置：x 前后偏移 ±0.08 m，y=0（中间），z 接地 -->
-            <origin xyz="${half_length - 0.032} ${(half_width - 0.0427) * flag} ${small_joint_z}" rpy="0 0 0" />
+            <origin xyz="${chassis_center_x + half_length - 0.032} ${(half_width - 0.0427) * flag} ${small_joint_z}" rpy="0 0 0" />
             <axis xyz="0 1 0" />                                 <!-- 绕 Y 轴旋转（球体无所谓） -->
         </joint>

File: src/mycar_description/urdf/car_laser.urdf.xacro (robot description, xacro)
@@ -14,10 +14,14 @@
     <!-- ================= 关节位置计算（相对于父坐标系） ================= -->
     <!-- 注意：以下计算用到了外部属性 base_length（车体高度），该属性需在调用此文件之前定义。 -->
-    <!-- 支撑柱关节在X轴上的偏移量（通常居中，故为0） -->
-    <xacro:property name="joint_support_x" value="0.07006" />
+    <!--
+      该数值描述激光雷达安装柱，不是托物转盘 support_link。旧模型中的
+      70.06 mm 以车体几何中心为基准；base_link 改到驱动轮轴中点后需加上
+      chassis_center_x，保持雷达的实体位置不变。
+    -->
+    <xacro:property name="joint_support_x" value="${chassis_center_x + 0.07006}" />
     <!-- 支撑柱关节在Y轴上的偏移量（通常居中，故为0） -->
     <xacro:property name="joint_support_y" value="0" />
     <!-- 支撑柱关节在Z轴上的偏移量：
-         从 base_link 的原点（一般为车体几何中心）出发，需要向上移动的距离。
+         从 base_link 的竖直参考高度出发，需要向上移动的距离。
          计算公式：车体半高（base_height/2） + 支撑柱半长（support_length/2）
          使得支撑柱的底部刚好接触车体顶部，且支撑柱的中心位于此高度。 -->
